File: mainBoard/mainBoard.kicad_pcb (KiCad board)
At the start: 2 copper layers, 92 x 61.9 mm, 60 parts, among them J1 program, J2 uniwersal-board2, SW1 reset, U1 STM32F407VGTx, U2 SMF05C / MMQA5V6T3G, U3 usb-micro, U4 MIC5504-3.3YM5, Y1 32kHz, Y2 8/16MHz

Commit message: Bug-fixes. 3 battery soldered and working.
Parts:
- JP4: value consoleTx -> consoleRx
- JP6: value consoleRx -> consoleTx
Connections:
- J1 pad 5: /consoleRx -> /consoleTx
- J1 pad 6: /consoleTx -> /consoleRx
- JP4 pad 1: /consoleTx -> /consoleRx
- JP6 pad 1: /consoleRx -> /consoleTx
- R10 pad 1: /swdclk -> /swdio
- R9 pad 1: /swdio -> /swdclk
Routing:
- net /swdclk: track 27.0 -> 24.4 mm
- net /swdio: track 27.7 -> 29.8 mm
- net /consoleTx: track 3.72 -> 3.03 mm
- net /consoleRx: track 3.03 -> 3.72 mm
- net /pa8: track 22.5 -> 23.1 mm
